File: kicad/RetroWiFiModem.sch (KiCad schematic (older format))
At the start: 32 parts, among them CON1 BARREL_JACK, P1 CONN_02X05, U1 74HCT245, U2 MAX3232, U3 74HC32, U4 LP2950ACZ-3.3, U5 WeMos_D1_mini

Commit message: update symbols and footprints for KiCad 5.1.2
* remaps all symbols and footprints to those present in KiCad 5.1.2.
* add mounting holes to schematics
* PCB has been touched up due to footprint changes, but should remain
  almost identical to the original
* NOTE: schematic now has some warnings about tristate<->output connections

symbols and footprints are mapped as follows:

Designator	Old symbol	Old package	New symbol	New package
C1,C2,C3,C4,C5,C8	C_Small	Capacitors_THT:C_Disc_D3_P2.5	Device:C_Small	Capacitor_THT:C_Disc_D3.0mm_W2.0mm_P2.50mm
C6	C_Small	Capacitors_THT:C_Disc_D3_P5	Device:C_Small	Capacitor_THT:C_Disc_D3.0mm_W2.0mm_P2.50mm
C7	C_Small	Capacitors_THT:C_Disc_D3_P2.5	Device:C_Small	Capacitor_THT:C_Disc_D3.0mm_W2.0mm_P2.50mm
CON1	BARREL_JACK	Connectors:BARREL_JACK	Connector:Barrel_Jack_Switch	Connector_BarrelJack:BarrelJack_Horizontal
D1,D2,D3,D4,D5,D6,D7,D8	LED	LEDs:LED-3MM	Device:LED	LED_THT:LED_D3.0mm
P1	CONN_02X05	Connectors:IDC_Header_Straight_10pins	Conn_02x05_Odd_Even	Connector_IDC:IDC-Header_2x05_P2.54mm_Vertical
U2	MAX232	Housings_DIP:DIP-16_W7.62mm	Interface_UART:MAX232	Package_DIP:DIP-16_W7.62mm
U3	74LS32	Housings_DIP:DIP-14_W7.62mm	74xx:74LS32	Package_DIP:DIP-14_W7.62mm
U4	LM2931AZ-3.3/5.0	TO_SOT_Packages_THT:TO-92_Inline_Wide	Regulator_Linear:LP2950-3.3_TO92	Package_TO_SOT_THT:TO-92L_Inline_Wide
U5	WeMos_mini	WEMOS_D1_Mini:wemos-d1-mini-with-pin-header-and-connector	RetroWiFiModem:WeMos_mini	footprint:wemos-d1-mini
U1	74ACT245	Housings_DIP:DIP-20_W7.62mm	74xx:74HC245	Package_DIP:DIP-20_W7.62mm
R1,R2,R3,R4,R5,R6,R7,R8	R_US	Discret:R3	Device:R	Resistor_THT:R_Axial_DIN0204_L3.6mm_D1.6mm_P7.62mm_Horizontal
R9	R_US	Discret:R3	Device:R	Resistor_THT:R_Axial_DIN0204_L3.6mm_D1.6mm_P7.62mm_Horizontal
H1,H2,H3,H4,H5,H6		Mounting_Holes:MountingHole_3.2mm_Hammond_1593	Mechanical:MountingHole	MountingHole:MountingHole_3.2mm_M3
Parts:
- removed U1: 74HCT245, Housings_DIP:DIP-20_W7.62mm, symbol 74ACT245
- added H1, H2, H3, H4, H5, H6: MountingHole, MountingHole:MountingHole_3.2mm_M3, symbol Mechanical:MountingHole
- added U1: 74HC245, Package_DIP:DIP-20_W7.62mm, symbol 74xx:74HC245
- added unit 5 of U3
- C1, C2, C3, C4, C5, C7, C8: footprint Capacitors_THT:C_Disc_D3_P2.5 -> Capacitor_THT:C_Disc_D3.0mm_W2.0mm_P2.50mm; symbol C_Small -> Device:C_Small
- C6: footprint Capacitors_THT:C_Disc_D3_P5 -> Capacitor_THT:C_Disc_D5.0mm_W2.5mm_P5.00mm; symbol C_Small -> Device:C_Small
- CON1: footprint Connectors:BARREL_JACK -> Connector_BarrelJack:BarrelJack_Horizontal; symbol BARREL_JACK -> Connector:Barrel_Jack_Switch
- D1, D2, D3, D4, D5, D6, D7, D8: footprint LEDs:LED-3MM -> LED_THT:LED_D3.0mm; symbol LED -> Device:LED
- P1: footprint Connectors:IDC_Header_Straight_10pins -> Connector_IDC:IDC-Header_2x05_P2.54mm_Vertical; symbol CONN_02X05 -> Connector_Generic:Conn_02x05_Odd_Even
- R1, R2, R3, R4, R5, R6, R7, R8, R9: footprint Discret:R3 -> Resistor_THT:R_Axial_DIN0204_L3.6mm_D1.6mm_P7.62mm_Horizontal; symbol R_US -> Device:R
- U2: footprint Housings_DIP:DIP-16_W7.62mm -> Package_DIP:DIP-16_W7.62mm; symbol MAX232 -> Interface_UART:MAX232
- U3: footprint Housings_DIP:DIP-14_W7.62mm -> Package_DIP:DIP-14_W7.62mm; symbol 74LS32 -> 74xx:74LS32
- U4: footprint TO_SOT_Packages_THT:TO-92_Inline_Wide -> Package_TO_SOT_THT:TO-92L_Inline_Wide; symbol LM2931AZ-3.3/5.0 -> Regulator_Linear:LP2950-3.3_TO92
- U5: footprint WEMOS_D1_Mini:wemos-d1-mini-with-pin-header-and-connector -> RetroWiFiModem-footprints:wemos-d1-mini; symbol WeMos_mini -> RetroWiFiModem:WeMos_mini
Connections:
- net +3V3: now also U3.14 (VCC); no longer U3.14 (VCC), U3.14 (VCC), U3.14 (VCC), U3.14 (VCC)
- net +5V: now also U1.20 (VCC)
- net GND: now also U1.1 (A->B), U1.10 (GND), U1.12 (B6), U1.19 (CE), U3.7 (GND); no longer U3.7 (GND), U3.7 (GND), U3.7 (GND), U3.7 (GND)
- net at U5.13 (D6): now also U1.15 (B3)
- net at U2.9 (R2OUT), U5.14 (D7): now also U1.18 (B0)
- net at U2.10 (T2IN), U5.15 (D8): now also U1.17 (B1)
- net at U5.5 (D2): now also U1.11 (B7)
- net at U5.6 (D1): now also U1.16 (B2)
- net at U2.12 (R1OUT), U5.7 (Rx): now also U1.13 (B5)
- net at U2.11 (T1IN), U3.3: now also U1.14 (B4)
- net at R1.1: now also U1.2 (A0)
- net at R2.1: now also U1.3 (A1)
- net at R3.1: now also U1.4 (A2)
- net at R4.1: now also U1.5 (A3)
- net at R5.1: now also U1.6 (A4)
- net at R6.1: now also U1.7 (A5)
- net at R7.1: now also U1.8 (A6)
- net at R8.1: now also U1.9 (A7)
Other:
- moved on the sheet: C5
